File: Arduino/PCB/ArduinoRgbFanController.sch (EAGLE design)
At the start: 53 parts, among them IC2 ARDUINO_MKRFOX1200PROTOPADS, Q1 MOSFET-PCHANNEL, Q2 MOSFET-NCHANNELAO3404A

Commit message: Tidied up schematic.
Added values to resistors.
Parts:
- R10, R7, R8, R9: value (none) -> 10k
- R2, R20, R3, R4, R6: value (none) -> 100k
- R21: value (none) -> 10R
- R28: value (none) -> 300R
- R5: value (none) -> 00k
Other:
- note added: "1.0"
- note added: "Connect for Internal"
- note added: "External 5V"
- note added: "External/Internal LED supply option"
- note added: "Stephen Harrison"
- note removed: "2"
- note removed: "S.Harrison"
- moved on the sheet: BME280, BME680, C1, C2, C3, C4, C5, C6, C7, D1, D2, D3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

Commit message: Updated to add dust sensor and switch/led drivers. Updated files at DirtyPCBs
Parts:
- added JP3: (no value), SparkFun-Connectors:M05PTH
- added JP5: (no value), SparkFun-Connectors:M03POLAR
- added R12, R13: 100k, SparkFun-Resistors:RESISTOR1206
- added R14, R15: 100R, SparkFun-Resistors:RESISTOR1206
- added R16: 10k, SparkFun-Resistors:RESISTOR1206
- added R17: 16k, SparkFun-Resistors:RESISTOR1206
- R5: value 00k -> 100k
Connections:
- net A6C renamed SWITCH_ENABLE
- removed net A2C: IC2.A2
- removed net A3C: IC2.A3
- removed net A4C: IC2.A4
- removed net A5C: IC2.A5
- new net LED1: IC2.A4, R14.2
- new net LED2: IC2.A5, R15.2
- new net N$3: JP3.3, R14.1
- new net N$4: JP3.2, R15.1
- new net N$7: JP5.2, R16.2
- new net SWITCH1: IC2.A2, JP3.5, R12.2
- new net SWITCH2: IC2.A3, JP3.4, R13.2
- net 3.3V: now also R12.1, R13.1
- net GND: now also JP3.1, JP5.1, R17.1
- net RXC: now also R16.1, R17.2
- net VIN: now also JP5.3
Other:
- note added: "Dust Sensor"
- note added: "Switches / LEDs"

Commit message: Moved dust sensor connection to PCB edge.
Removed pullup/down resistors for PWM and tach signals as they are not needed.

Added P-FET + N-FET power control to switch the 12V to the PWM fans as some fans do not switch off when PWM off.

Moved 12V LED to switched fan power line and to underneath the "On" lettering.
Parts:
- removed R10, R7, R8, R9: 10k, SparkFun-Resistors:RESISTOR1206
- removed R2, R3, R4, R5, R6: 100k, SparkFun-Resistors:RESISTOR1206
- added Q3: 2N7002, SparkFun-DiscreteSemi:MOSFET-NCHANNELAO3404A
- added Q4: IRLML9301TRPBF, SparkFun-DiscreteSemi:MOSFET-PCHANNEL
- added R18: 10R, SparkFun-Resistors:RESISTOR0805-RES
- added R19: 100k, SparkFun-Resistors:RESISTOR0805-RES
- added R22, R23: 1M, SparkFun-Resistors:RESISTOR0805-RES
- Q1: value MOSFET-PCHANNEL -> IRLML9301TRPBF
- Q2: value MOSFET-NCHANNELAO3404A -> 2N7002
- R1, R11, R12, R13, R14, R15, R16, R17, R20, R21: device SparkFun-Resistors:RESISTOR1206 -> SparkFun-Resistors:RESISTOR0805-RES
Connections:
- removed net MISO: IC2.MISO
- removed net RXC: IC2.RX, R16.1, R17.2
- removed net SWITCH_ENABLE: IC2.A6
- new net DUST_SENSOR: IC2.D6, R16.1, R17.2
- new net FAN_POWER: JP13.2, JP6.2, JP8.2, JP9.2, Q1.S, Q4.D, R20.2, R28.1
- new net FAN_POWER_CONTROL: IC2.RX, R18.2, R22.1
- new net N$5: Q3.D, Q4.G, R19.2
- new net N$6: Q3.G, R18.1
- new net SWITCH_ENABLED: IC2.A5
- net 12V: now also Q4.S, R19.1; no longer JP13.2, JP6.2, JP8.2, JP9.2, Q1.S, R20.2, R28.1
- net 3.3V: no longer C6.1, R2.1, R3.1, R4.1, R5.1, R6.1
- net FAN1_PWM: no longer R10.1
- net FAN1_TACH: no longer R2.2
- net FAN2_PWM: no longer R9.1
- net FAN2_TACH: no longer R3.2
- net FAN3_PWM: no longer R8.1
- net FAN3_TACH: no longer R4.2
- net FAN4_PWM: no longer R7.1
- net FAN4_TACH: no longer R5.2
- net FAN5_PWM: now also IC2.MISO, R23.1; no longer IC2.D6
- net FAN5_TACH: no longer R6.2
- net GND: now also Q3.S, R22.2, R23.2; no longer R10.2, R7.2, R8.2, R9.2
- net LED2: now also IC2.A3; no longer IC2.A5
- net N$3: now also JP3.2; no longer JP3.3
- net N$4: now also JP3.3; no longer JP3.2
- net OSH_LED: now also IC2.A6; no longer IC2.A1
- net SWITCH1: now also JP3.4; no longer JP3.5
- net SWITCH2: now also IC2.A1, JP3.5; no longer IC2.A3, JP3.4
- net VIN: now also C6.1
Other:
- moved on the sheet: C6, R14, R15
